Commit message: add abs pose publisher and fix pivoting joint

File: dual_arm_control/urdf/iiwa_ibr_pivoting.xacro (robot description, xacro)
@@ -10,9 +10,9 @@
   <link name="$(arg prefix)pivoting_link" />
 <joint name="$(arg prefix)pivoting_joint" type="revolute" >
-    <origin xyz="0.0 0 0.2" rpy="0 0 0"/>
+    <origin xyz="0.0 0 0.2" rpy="1.57079637 0 0"/>
     <parent link="$(arg prefix)link8" />
     <child link="$(arg prefix)pivoting_link" />
     <limit effort="0" lower="-1.57079637" upper="1.57079637" velocity="6.10865255"/>
-    <axis xyz="0 1 0"/>
+    <axis xyz="0 0 1"/>
 </joint>
 </robot>

File: dual_arm_control/urdf/sia5d_pivoting.xacro (robot description, xacro)
@@ -7,9 +7,9 @@
 	<link name="$(arg prefix)pivoting_link" />
 	<joint name="$(arg prefix)pivoting_joint" type="revolute" >
-		<origin xyz="0.0 0 0.2" rpy="0 0 0"/>
+		<origin xyz="0.0 0 0.2" rpy="1.57079637 0 0"/>
 		<parent link="$(arg prefix)tool0" />
 		<child link="$(arg prefix)pivoting_link" />
 		<limit effort="0" lower="-1.57079637" upper="1.57079637" velocity="6.10865255"/>
-		<axis xyz="0 1 0"/>
+		<axis xyz="0 0 -1"/>
 	</joint>
 </robot>

Commit message: add joint mux/demux, fix DH iiwa pivoting, to fix camera iiwa transform

File: dual_arm_control/urdf/iiwa_ibr_pivoting.xacro (robot description, xacro)
@@ -10,5 +10,5 @@
   <link name="$(arg prefix)pivoting_link" />
 <joint name="$(arg prefix)pivoting_joint" type="revolute" >
-    <origin xyz="0.0 0 0.2" rpy="1.57079637 0 0"/>
+    <origin xyz="0.0 0 0.2" rpy="1.57079637 0 1.57079637"/>
     <parent link="$(arg prefix)link8" />
     <child link="$(arg prefix)pivoting_link" />
