Commit message: add urdf pivoting iiwa

File: dual_arm_control/urdf/sia5d_pivoting.xacro (robot description, xacro)
@@ -2,11 +2,12 @@
 <!--Generates a urdf from the macro in sia5_macro.xacro -->
 <robot name="motoman_sia5d" xmlns:xacro="http://ros.org/wiki/xacro">
+    <xacro:arg name="prefix" default="yaskawa_"/>
 	<xacro:include filename="$(find uclv_robot_ros)/urdf/robots/motoman_sia5f/sia5d_macro.xacro"/>
-	<xacro:motoman_sia5d prefix=""/>
-	<link name="pivoting_link" />
-	<joint name="tool0-pivoting_link" type="revolute" >
+	<xacro:motoman_sia5d prefix="$(arg prefix)"/>
+	<link name="$(arg prefix)pivoting_link" />
+	<joint name="$(arg prefix)pivoting_joint" type="revolute" >
 		<origin xyz="0.0 0 0.2" rpy="0 0 0"/>
-		<parent link="tool0" />
-		<child link="pivoting_link" />
+		<parent link="$(arg prefix)tool0" />
+		<child link="$(arg prefix)pivoting_link" />
 		<limit effort="0" lower="-1.57079637" upper="1.57079637" velocity="6.10865255"/>
 		<axis xyz="0 1 0"/>

Commit message: minor fix

File: dual_arm_control/urdf/sia5d_pivoting.xacro (robot description, xacro)
@@ -7,5 +7,5 @@
 	<link name="$(arg prefix)pivoting_link" />
 	<joint name="$(arg prefix)pivoting_joint" type="revolute" >
-		<origin xyz="0.0 0 0.2" rpy="1.57079637 0 0"/>
+		<origin xyz="0.0 0 0.178" rpy="1.57079637 0 0"/>
 		<parent link="$(arg prefix)tool0" />
 		<child link="$(arg prefix)pivoting_link" />
